File: hardware/Ornament.kicad_pcb (KiCad board)
At the start: 2 copper layers, 93.6 x 101.9 mm, 37 parts, among them J1 SWDIO, Q1 HL3400, Q2 HL3400, SW1 HX 0805-C2, U1 PY32F002BL15S7TU

Commit message: add silk text
Parts:
- moved BT1 1.52 mm to (146.4, 105.2)
Other:
- board text added: "From: Jacob, Sasha Zhuzhu, & Wormy"
- board text added: "Happy Holidays!"

Commit message: Update Ornament.kicad_pcb
Other:
- board text added: "From: Jacob, Sasha, Zhuzhu, & Wormy"
- board text added: "Ornament2026 Rev0"
- board text removed: "From: Jacob, Sasha Zhuzhu, & Wormy"
Changed lines of the file:
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@@
 		)
 	)
-	(gr_text "From:\nJacob, Sasha\nZhuzhu, & Wormy"
+	(gr_text "Ornament2026\nRev0"
+		(at 138.2776 140.5636 70)
+		(layer "B.SilkS")
+		(effects
+			(font
+				(size 1 1)
+				(thickness 0.1)
+			)
+			(justify left bottom mirror)
+		)
+	)
+	(gr_text "From:\nJacob, Sasha,\nZhuzhu, & Wormy"
 		(at 148.7046 116.7826 0)
 		(layer "B.SilkS")

Commit message: update SWD connector
Parts:
- J1: moved to B.Cu
- R1, R10, R11, R12, R13, R14, R15, R2, R3, R4, R5, R6, R7, R8, R9: value 47 -> 150
- moved J1 24.2 mm to (125.7, 103.2), turned to 90 degrees
Connections:
- J1 pad 1: /SWDIO -> +3V
- J1 pad 2: GND -> /SWDIO
Routing:
- net /SWDIO: track 2.58 -> 29.6 mm, vias 0 -> 1
- net /SWCLK: track 2.58 -> 24.2 mm, vias 0 -> 1
- net GND: track 8.21 -> 6.43 mm, vias 5 -> 4
- net +3V: track 3.80 -> 5.58 mm, vias 3 -> 4
