File: hardware/Ornament.kicad_pcb (KiCad board)
At the start: 2 copper layers, 93.6 x 101.9 mm, 37 parts, among them J1 SWDIO, Q1 HL3400, Q2 HL3400, SW1 HX 0805-C2, U1 PY32F002BL15S7TU

Commit message: update CR2032 holder MPN
Parts:
- BT1: value CR2032-BS-6-1 -> A-BAT-CH-C8-EA-ZSR3
Changed lines of the file:
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@@
 			)
 		)
-		(attr smd)
+		(attr smd exclude_from_bom)
 		(duplicate_pad_numbers_are_jumpers no)
 		(fp_text user "${REFERENCE}"
@@
 			)
 		)
-		(property "Value" "CR2032-BS-6-1"
+		(property "Value" "A-BAT-CH-C8-EA-ZSR3"
 			(at 0 -1 0)
 			(unlocked yes)
@@
 			)
 		)
-		(property "Datasheet" "https://www.lcsc.com/product-detail/C70377.html"
+		(property "Datasheet" "https://mm.digikey.com/Volume0/opasdata/d220001/medias/docus/6167/A-BAT-CH-C8-EA-ZSR3.PDF"
 			(at 0 0 0)
 			(unlocked yes)
@@
 			)
 		)
-		(property "JLCPCB Part Number" "C70377"
+		(property "JLCPCB Part Number" ""
 			(at 0 0 0)
 			(unlocked yes)
@@
 			)
 		)
-		(attr smd)
+		(attr smd exclude_from_bom)
 		(duplicate_pad_numbers_are_jumpers no)
 		(fp_line
@@
 	)
 	(segment
-		(start 148.6916 106.7816)
-		(end 148.9456 106.7816)
-		(width 0.2)
-		(layer "F.Cu")
-		(net "/SWDIO")
-	)
-	(segment
-		(start 150.5966 105.1306)
-		(end 151.6101 105.1306)
-		(width 0.2)
-		(layer "F.Cu")
-		(net "/SWDIO")
-	)
-	(segment
-		(start 148.9456 106.7816)
-		(end 150.5966 105.1306)
-		(width 0.2)
-		(layer "F.Cu")
-		(net "/SWDIO")
-	)
-	(via
-		(at 148.6916 106.7816)
-		(size 0.45)
-		(drill 0.3)
-		(layers "F.Cu" "B.Cu")
-		(net "/SWDIO")
-	)
-	(segment
-		(start 127.7386 106.7816)
-		(end 148.6916 106.7816)
-		(width 0.2)
-		(layer "B.Cu")
-		(net "/SWDIO")
-	)
-	(segment
-		(start 124.1826 103.2256)
-		(end 127.7386 106.7816)
-		(width 0.2)
-		(layer "B.Cu")
-		(net "/SWDIO")
-	)
-	(segment
-		(start 150.3426 101.3206)
-		(end 149.7076 101.9556)
-		(width 0.2)
-		(layer "F.Cu")
-		(net "GND")
-	)
-	(segment
-		(start 157.1521 101.3816)
-		(end 157.1521 102.4151)
-		(width 0.2)
-		(layer "F.Cu")
-		(net "GND")
-	)
-	(segment
-		(start 141.3256 105.7656)
-		(end 141.3256 107.3931)
-		(width 0.2)
-		(layer "F.Cu")
-		(net "GND")
-	)
-	(segment
-		(start 157.1521 102.4151)
-		(end 157.2006 102.4636)
-		(width 0.2)
-		(layer "F.Cu")
-		(net "GND")
-	)
-	(segment
-		(start 151.5466 95.4001)
-		(end 151.5466 96.3016)
-		(width 0.2)
-		(layer "F.Cu")
-		(net "GND")
-	)
-	(segment
-		(start 151.6101 101.3206)
-		(end 150.3426 101.3206)
-		(width 0.2)
-		(layer "F.Cu")
-		(net "GND")
-	)
-	(segment
-		(start 151.5466 96.3016)
-		(end 151.9936 96.7486)
-		(width 0.2)
-		(layer "F.Cu")
-		(net "GND")
-	)
-	(via
-		(at 157.2006 102.4636)
-		(size 0.45)
-		(drill 0.3)
-		(layers "F.Cu" "B.Cu")
-		(net "GND")
-	)
-	(via
-		(at 141.3256 107.3931)
-		(size 0.45)
-		(drill 0.3)
-		(layers "F.Cu" "B.Cu")
-		(net "GND")
-	)
-	(via
-		(at 151.9936 96.7486)
-		(size 0.45)
-		(drill 0.3)
-		(layers "F.Cu" "B.Cu")
-		(net "GND")
-	)
-	(via
-		(at 149.7076 101.9556)
-		(size 0.45)
-		(drill 0.3)
-		(layers "F.Cu" "B.Cu")
-		(net "GND")
-	)
-	(segment
-		(start 144.7546 105.1306)
-		(end 146.5351 105.1306)
-		(width 0.2)
-		(layer "F.Cu")
-		(net "/SWCLK")
-	)
-	(via
-		(at 144.7546 105.1306)
-		(size 0.45)
-		(drill 0.3)
-		(layers "F.Cu" "B.Cu")
-		(net "/SWCLK")
-	)
-	(segment
-		(start 124.1826 100.6856)
-		(end 128.6276 105.1306)
-		(width 0.2)
-		(layer "B.Cu")
-		(net "/SWCLK")
-	)
-	(segment
-		(start 128.6276 105.1306)
-		(end 144.7546 105.1306)
-		(width 0.2)
-		(layer "B.Cu")
-		(net "/SWCLK")
-	)
-	(segment
 		(start 122.4026 61.9506)
 		(end 116.8146 67.5386)
@@
 	)
 	(segment
+		(start 144.7546 105.1306)
+		(end 146.5351 105.1306)
+		(width 0.2)
+		(layer "F.Cu")
+		(net "/SWCLK")
+	)
+	(via
+		(at 144.7546 105.1306)
+		(size 0.45)
+		(drill 0.3)
+		(layers "F.Cu" "B.Cu")
+		(net "/SWCLK")
+	)
+	(segment
+		(start 124.1826 100.6856)
+		(end 128.6276 105.1306)
+		(width 0.2)
+		(layer "B.Cu")
+		(net "/SWCLK")
+	)
+	(segment
+		(start 128.6276 105.1306)
+		(end 144.7546 105.1306)
+		(width 0.2)
+		(layer "B.Cu")
+		(net "/SWCLK")
+	)
+	(segment
+		(start 148.6916 106.7816)
+		(end 148.9456 106.7816)
+		(width 0.2)
+		(layer "F.Cu")
+		(net "/SWDIO")
+	)
+	(segment
+		(start 150.5966 105.1306)
+		(end 151.6101 105.1306)
+		(width 0.2)
+		(layer "F.Cu")
+		(net "/SWDIO")
+	)
+	(segment
+		(start 148.9456 106.7816)
+		(end 150.5966 105.1306)
+		(width 0.2)
+		(layer "F.Cu")
+		(net "/SWDIO")
+	)
+	(via
+		(at 148.6916 106.7816)
+		(size 0.45)
+		(drill 0.3)
+		(layers "F.Cu" "B.Cu")
+		(net "/SWDIO")
+	)
+	(segment
+		(start 127.7386 106.7816)
+		(end 148.6916 106.7816)
+		(width 0.2)
+		(layer "B.Cu")
+		(net "/SWDIO")
+	)
+	(segment
+		(start 124.1826 103.2256)
+		(end 127.7386 106.7816)
+		(width 0.2)
+		(layer "B.Cu")
+		(net "/SWDIO")
+	)
+	(segment
 		(start 151.6101 102.5906)
 		(end 154.0431 102.5906)
@@
 	)
 	(segment
+		(start 150.3426 101.3206)
+		(end 149.7076 101.9556)
+		(width 0.2)
+		(layer "F.Cu")
+		(net "GND")
+	)
+	(segment
+		(start 157.1521 101.3816)
+		(end 157.1521 102.4151)
+		(width 0.2)
+		(layer "F.Cu")
+		(net "GND")
+	)
+	(segment
+		(start 141.3256 105.7656)
+		(end 141.3256 107.3931)
+		(width 0.2)
+		(layer "F.Cu")
+		(net "GND")
+	)
+	(segment
+		(start 157.1521 102.4151)
+		(end 157.2006 102.4636)
+		(width 0.2)
+		(layer "F.Cu")
+		(net "GND")
+	)
+	(segment
+		(start 151.5466 95.4001)
+		(end 151.5466 96.3016)
+		(width 0.2)
+		(layer "F.Cu")
+		(net "GND")
+	)
+	(segment
+		(start 151.6101 101.3206)
+		(end 150.3426 101.3206)
+		(width 0.2)
+		(layer "F.Cu")
+		(net "GND")
+	)
+	(segment
+		(start 151.5466 96.3016)
+		(end 151.9936 96.7486)
+		(width 0.2)
+		(layer "F.Cu")
+		(net "GND")
+	)
+	(via
+		(at 157.2006 102.4636)
+		(size 0.45)
+		(drill 0.3)
+		(layers "F.Cu" "B.Cu")
+		(net "GND")
+	)
+	(via
+		(at 141.3256 107.3931)
+		(size 0.45)
+		(drill 0.3)
+		(layers "F.Cu" "B.Cu")
+		(net "GND")
+	)
+	(via
+		(at 151.9936 96.7486)
+		(size 0.45)
+		(drill 0.3)
+		(layers "F.Cu" "B.Cu")
+		(net "GND")
+	)
+	(via
+		(at 149.7076 101.9556)
+		(size 0.45)
+		(drill 0.3)
+		(layers "F.Cu" "B.Cu")
+		(net "GND")
+	)
+	(segment

Commit message: update silk
Parts:
- moved Q2 2.80 mm to (158.0, 103.2)
Routing:
- net /LED_B1: track 6.83 -> 5.55 mm
- net GND: track 6.43 -> 7.12 mm
Other:
- board text added: "GND"
- board text added: "SWCLK"
- board text added: "SWDIO"
- board text added: "VCC"
Changed lines of the file:
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@@
 	(footprint "Package_TO_SOT_SMD:SOT-23"
 		(layer "F.Cu")
-		(at 158.0896 100.4316)
+		(at 157.9626 103.2256)
 		(descr "SOT, 3 Pin (JEDEC TO-236 Var AB https://www.jedec.org/document_search?search_api_views_fulltext=TO-236)")
 		(tags "SOT TO_SOT_SMD")
@@
 		(layer "Edge.Cuts")
 	)
-	(gr_text "Happy\nHolidays!"
-		(at 165.9456 103.701404 0)
-		(layer "F.SilkS")
+	(gr_text "Ornament2026\nRev0"
+		(at 138.2776 140.5636 70)
+		(layer "B.SilkS")
 		(effects
 			(font
-				(size 2.54 2.54)
-				(bold yes)
+				(size 1 1)
+				(thickness 0.1)
 			)
+			(justify left bottom mirror)
 		)
 	)
-	(gr_text "Ornament2026\nRev0"
-		(at 138.2776 140.5636 70)
+	(gr_text "GND"
+		(at 128.7526 98.7806 0)
 		(layer "B.SilkS")
 		(effects
 			(font
 				(size 1 1)
-				(thickness 0.1)
+				(thickness 0.15)
+			)
+			(justify left bottom mirror)
+		)
+	)
+	(gr_text "VCC"
+		(at 128.7526 106.4006 0)
+		(layer "B.SilkS")
+		(effects
+			(font
+				(size 1 1)
+				(thickness 0.15)
 			)
 			(justify left bottom mirror)
 		)
 	)
-	(gr_text "From:\nJacob, Sasha,\nZhuzhu, & Wormy"
-		(at 148.7046 116.7826 0)
+	(gr_text "SWDIO"
+		(at 130.4036 103.8606 0)
+		(layer "B.SilkS")
+		(effects
+			(font
+				(size 1 1)
+				(thickness 0.15)
+			)
+			(justify left bottom mirror)
+		)
+	)
+	(gr_text "SWCLK"
+		(at 130.6576 101.3206 0)
+		(layer "B.SilkS")
+		(effects
+			(font
+				(size 1 1)
+				(thickness 0.15)
+			)
+			(justify left bottom mirror)
+		)
+	)
+	(gr_text "From: Jacob,\nSasha, Zhuzhu,\n& Wormy"
+		(at 148.844 116.84 0)
+		(layer "B.SilkS")
+		(effects
+			(font
+				(size 1.524 1.524)
+				(bold yes)
+			)
+			(justify top mirror)
+		)
+	)
+	(gr_text "Happy Holidays!\n"
+		(at 148.844 113.66629 0)
 		(layer "B.SilkS")
 		(effects
@@
 	)
 	(segment
+		(start 154.3581 102.2756)
+		(end 157.0251 102.2756)
+		(width 0.2)
+		(layer "F.Cu")
+		(net "/LED_B1")
+	)
+	(segment
 		(start 151.6101 102.5906)
 		(end 154.0431 102.5906)
@@
 	(segment
 		(start 154.0431 102.5906)
-		(end 157.1521 99.4816)
+		(end 154.3581 102.2756)
 		(width 0.2)
 		(layer "F.Cu")
@@
 	)
 	(segment
-		(start 150.3426 101.3206)
-		(end 149.7076 101.9556)
+		(start 155.9306 105.5116)
+		(end 157.0251 104.4171)
 		(width 0.2)
 		(layer "F.Cu")
@@
 	)
 	(segment
-		(start 157.1521 101.3816)
-		(end 157.1521 102.4151)
+		(start 150.3426 101.3206)
+		(end 149.7076 101.9556)
 		(width 0.2)
 		(layer "F.Cu")
@@
 	)
 	(segment
-		(start 157.1521 102.4151)
-		(end 157.2006 102.4636)
+		(start 157.0251 104.4171)
+		(end 157.0251 104.1756)
 		(width 0.2)
 		(layer "F.Cu")
@@
 	)
 	(via
-		(at 157.2006 102.4636)
+		(at 155.9306 105.5116)
 		(size 0.45)
 		(drill 0.3)
