File: hardware/Ornament.kicad_sch (KiCad schematic)
At the start: 37 parts, among them J1 SWDIO, Q1 HL3400, Q2 HL3400, SW1 HX 0805-C2, U1 PY32F002BL15S7TU

Commit message: init dev board
Parts:
- D1, D10, D11, D12, D13, D14, D15, D2, D3, D4, D5, D6, D7, D8, D9: JLCPCB Part Number KT-0603W -> C2290
Changed lines of the file:
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@@
 			)
 		)
-		(property "JLCPCB Part Number" "KT-0603W"
+		(property "JLCPCB Part Number" "C2290"
 			(at 215.9 62.23 90)
 			(hide yes)
@@
 			)
 		)
-		(property "JLCPCB Part Number" "KT-0603W"
+		(property "JLCPCB Part Number" "C2290"
 			(at 254 113.03 90)
 			(hide yes)
@@
 			)
 		)
-		(property "JLCPCB Part Number" "KT-0603W"
+		(property "JLCPCB Part Number" "C2290"
 			(at 139.7 113.03 90)
 			(hide yes)
@@
 			)
 		)
-		(property "JLCPCB Part Number" "KT-0603W"
+		(property "JLCPCB Part Number" "C2290"
 			(at 196.85 62.23 90)
 			(hide yes)
@@
 			)
 		)
-		(property "JLCPCB Part Number" "KT-0603W"
+		(property "JLCPCB Part Number" "C2290"
 			(at 234.95 113.03 90)
 			(hide yes)
@@
 			)
 		)
-		(property "JLCPCB Part Number" "KT-0603W"
+		(property "JLCPCB Part Number" "C2290"
 			(at 120.65 113.03 90)
 			(hide yes)
@@
 			)
 		)
-		(property "JLCPCB Part Number" "KT-0603W"
+		(property "JLCPCB Part Number" "C2290"
 			(at 234.95 62.23 90)
 			(hide yes)
@@
 			)
 		)
-		(property "JLCPCB Part Number" "KT-0603W"
+		(property "JLCPCB Part Number" "C2290"
 			(at 139.7 62.23 90)
 			(hide yes)
@@
 			)
 		)
-		(property "JLCPCB Part Number" "KT-0603W"
+		(property "JLCPCB Part Number" "C2290"
 			(at 196.85 113.03 90)
 			(hide yes)
@@
 			)
 		)
-		(property "JLCPCB Part Number" "KT-0603W"
+		(property "JLCPCB Part Number" "C2290"
 			(at 158.75 62.23 90)
 			(hide yes)
@@
 			)
 		)
-		(property "JLCPCB Part Number" "KT-0603W"
+		(property "JLCPCB Part Number" "C2290"
 			(at 177.8 113.03 90)
 			(hide yes)
@@
 			)
 		)
-		(property "JLCPCB Part Number" "KT-0603W"
+		(property "JLCPCB Part Number" "C2290"
 			(at 177.8 62.23 90)
 			(hide yes)
@@
 			)
 		)
-		(property "JLCPCB Part Number" "KT-0603W"
+		(property "JLCPCB Part Number" "C2290"
 			(at 120.65 62.23 90)
 			(hide yes)
@@
 			)
 		)
-		(property "JLCPCB Part Number" "KT-0603W"
+		(property "JLCPCB Part Number" "C2290"
 			(at 215.9 113.03 90)
 			(hide yes)
@@
 			)
 		)
-		(property "JLCPCB Part Number" "KT-0603W"
+		(property "JLCPCB Part Number" "C2290"
 			(at 158.75 113.03 90)
 			(hide yes)
