File: hardware/Ornament.kicad_sch (KiCad schematic)
At the start: 37 parts, among them J1 SWDIO, Q1 HL3400, Q2 HL3400, SW1 HX 0805-C2, U1 PY32F002BL15S7TU

Commit message: update SWD connector
Parts:
- J1: symbol Connector:Conn_01x03_Socket -> Connector_Generic:Conn_01x04; now in the parts list
- R1, R10, R11, R12, R13, R14, R15, R2, R3, R4, R5, R6, R7, R8, R9: value 47 -> 150; JLCPCB Part Number C23182 -> C22808
Connections:
- net +3V: now also J1.1 (Pin_1)
- net GND: now also J1.4 (Pin_4); no longer J1.2 (Pin_2)
- net SWDIO: now also J1.2 (Pin_2); no longer J1.1 (Pin_1)

Commit message: update CR2032 holder MPN
Parts:
- BT1: value CR2032-BS-6-1 -> A-BAT-CH-C8-EA-ZSR3; JLCPCB Part Number C70377 -> (none); now left out of the parts list
- J1: now left out of the parts list
Changed lines of the file:
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@@
 		(body_style 1)
 		(exclude_from_sim no)
-		(in_bom yes)
+		(in_bom no)
 		(on_board yes)
 		(in_pos_files yes)
@@
 			)
 		)
-		(property "Value" "CR2032-BS-6-1"
+		(property "Value" "A-BAT-CH-C8-EA-ZSR3"
 			(at 54.61 51.4984 0)
 			(show_name no)
@@
 			)
 		)
-		(property "Datasheet" "https://www.lcsc.com/product-detail/C70377.html"
+		(property "Datasheet" "https://mm.digikey.com/Volume0/opasdata/d220001/medias/docus/6167/A-BAT-CH-C8-EA-ZSR3.PDF"
 			(at 50.8 50.546 90)
 			(hide yes)
@@
 			)
 		)
-		(property "JLCPCB Part Number" "C70377"
+		(property "JLCPCB Part Number" ""
 			(at 50.8 52.07 0)
 			(hide yes)
@@
 		(body_style 1)
 		(exclude_from_sim no)
-		(in_bom yes)
+		(in_bom no)
 		(on_board yes)
 		(in_pos_files yes)
